File: PCB/ProletarianPower_PedalPCB.kicad_sch (KiCad schematic)
At the start: 21 parts, among them J1 NJ2FD-V, J2 NJ2FD-V, U1 TL082

Commit message: completed schematic
Parts:
- added C10, C9: 1uF, Capacitor_THT:CP_Radial_D4.0mm_P2.00mm, symbol Device:C
- added C8: 220 nF, Capacitor_THT:CP_Radial_D4.0mm_P2.00mm, symbol Device:C
- added D3, D4: 1N4148, Diode_THT:D_DO-35_SOD27_P7.62mm_Horizontal, symbol Diode:1N4148
- added R10: 220, PCM_SparkFun-Resistor:R_Axial_DIN0207_L6.3mm_D2.5mm_P7.62mm_Horizontal, symbol PCM_SparkFun-Resistor:R
- added R6: 10k, PCM_SparkFun-Resistor:R_Axial_DIN0207_L6.3mm_D2.5mm_P7.62mm_Horizontal, symbol PCM_SparkFun-Resistor:10k_Axial_1/6W
- added R8, R9: 1k, PCM_SparkFun-Resistor:R_Axial_DIN0207_L6.3mm_D2.5mm_P7.62mm_Horizontal, symbol PCM_SparkFun-Resistor:R
- added SW2: SW_SPST, Connector_Wire:SolderWire-0.127sqmm_1x02_P3.7mm_D0.48mm_OD1mm, symbol Switch:SW_SPST
- added SW3: SW_DPDT_x2, Button_Switch_THT:SW_CK_JS202011CQN_DPDT_Straight, symbol Switch:SW_DPDT_x2
- added unit 2 of U1
- BT1: footprint (none) -> PCM_SparkFun-Connector:Barrel_Jack_PTH
- C0: renamed from C1; footprint PCM_SparkFun-Capacitor:Panasonic_D -> Capacitor_THT:CP_Radial_D4.0mm_P2.00mm
- C1: footprint (none) -> Capacitor_THT:CP_Radial_D5.0mm_P2.00mm
- C2: footprint PCM_SparkFun-Capacitor:Panasonic_D -> Capacitor_THT:CP_Radial_D4.0mm_P2.00mm
- C3, C4, C5: footprint (none) -> Capacitor_THT:CP_Radial_D4.0mm_P2.00mm
- C6: value 22 nF -> 220 nF; footprint (none) -> Capacitor_THT:CP_Radial_D4.0mm_P2.00mm
- R1, R2, R3, R4, R5: footprint PCM_SparkFun-Resistor:R_0603_1608Metric -> PCM_SparkFun-Resistor:R_Axial_DIN0207_L6.3mm_D2.5mm_P7.62mm_Horizontal
- RV1, RV3: footprint (none) -> Potentiometer_THT:Potentiometer_Alps_RK09K_Single_Vertical
- RV2: value 500k -> 20k; footprint (none) -> Potentiometer_THT:Potentiometer_Alps_RK09K_Single_Vertical
- U1: footprint (none) -> Package_DIP:SMDIP-8_W7.62mm
Connections:
- net GND: now also C6.1, D3.2 (A), D4.1 (K), R10.1; no longer C6.2
- net EFFECT_OUT: now reaches RV3.2
- net EFFECT_OUT: now also SW3.6 (C); no longer J2.T
- net at RV3.1: now also R8.2; no longer RV2.1
- net at RV2.2: now also C8.1; no longer C6.1
- net at C5.1, RV2.3: now also C6.2, C10.1, R6.1, U1.5 (+)
- net EFFECT_IN: now reaches R3.1
- net EFFECT_IN: now also SW3.3 (C); no longer J1.T
- net 4.5V: now reaches C1.1, R4.2, U1.3 (+)
- net 4.5V: now also R6.2
- new net: C8.2, R10.2
- new net: C9.2, R8.1
- new net: D3.1 (K), D4.2 (A), SW2.2 (B)
- new net: C10.2, SW2.1 (A)
- new net: C9.1, R9.2, U1.7
- new net: R9.1, RV2.1, U1.6 (-)
- new net INPUT: J1.T, SW3.2 (B), SW3.4 (A)
- new net OUTPUT: J2.T, SW3.1 (A), SW3.5 (B)
Other:
- note added: "HARD CLIPPING"
- note added: "i think it's 4.5V"
- note added: "input output"
- note added: "slightly better tone knob (thank you tube screamer)"
- note added: "toggle"
- note added: "volume + output"
- note removed: "INPUT"
- note removed: "variable low-pass filter (shitty tone knob)"
- moved on the sheet: BT1, C0, C2, J1, J2, R1, R2, R4, R5, RV3

Commit message: completed pcb
Parts:
- added H1, H2, H3, H4: MountingHole_Pad, MountingHole:MountingHole_3.2mm_M3_DIN965_Pad_TopBottom, symbol Mechanical:MountingHole_Pad
- C1: value C_Polarized_Small -> 470nF
- C10, C3, C4, C6, C8, C9: footprint Capacitor_THT:CP_Radial_D4.0mm_P2.00mm -> Capacitor_THT:C_Axial_L5.1mm_D3.1mm_P7.50mm_Horizontal
- C5: value C_Polarized_Small -> 1uF
- J1, J2: footprint Connector_Audio:Jack_6.35mm_Neutrik_NJ2FD-V_Vertical -> Connector_Audio:Jack_6.35mm_Neutrik_NMJ4HFD2_Horizontal
Connections:
- net GND: now also H1.1, H2.1, H3.1, H4.1
